Commit message: pr2 panda robotiq redone

File: pr2/pr2.urdf (robot description, URDF)
Before this commit: robot pr2, 82 links, 81 joints
Links:
- link base_link: geometry collision mesh filename=package://pr2_description/meshes/base_v0/base_L.stl; visual mesh filename=package://pr2_description/meshes/base_v0/base.stl scale=0.001 0.001 0.001

Commit message: urdf conversions redone

File: pr2/pr2.urdf (robot description, URDF)
Before this commit: robot pr2, 82 links, 81 joints
Links:
- link base_link: geometry collision mesh filename=package://pr2_description/meshes/base_v0/base_L.stl; visual mesh filename=package://pr2_description/meshes/base_v0/base.dae
- link bl_caster_l_wheel_link: geometry collision cylinder length=0.034 radius=0.074792; visual mesh filename=package://pr2_description/meshes/base_v0/wheel.dae
- link bl_caster_r_wheel_link: geometry collision cylinder length=0.034 radius=0.074792; visual mesh filename=package://pr2_description/meshes/base_v0/wheel.dae
- link br_caster_l_wheel_link: geometry collision cylinder length=0.034 radius=0.074792; visual mesh filename=package://pr2_description/meshes/base_v0/wheel.dae
- link br_caster_r_wheel_link: geometry collision cylinder length=0.034 radius=0.074792; visual mesh filename=package://pr2_description/meshes/base_v0/wheel.dae
- link fl_caster_l_wheel_link: geometry collision cylinder length=0.034 radius=0.074792; visual mesh filename=package://pr2_description/meshes/base_v0/wheel.dae
- link fl_caster_r_wheel_link: geometry collision cylinder length=0.034 radius=0.074792; visual mesh filename=package://pr2_description/meshes/base_v0/wheel.dae
- link fr_caster_l_wheel_link: geometry collision cylinder length=0.034 radius=0.074792; visual mesh filename=package://pr2_description/meshes/base_v0/wheel.dae
- link fr_caster_r_wheel_link: geometry collision cylinder length=0.034 radius=0.074792; visual mesh filename=package://pr2_description/meshes/base_v0/wheel.dae
- link head_pan_link: geometry collision mesh filename=package://pr2_description/meshes/head_v0/head_pan_L.stl; visual mesh filename=package://pr2_description/meshes/head_v0/head_pan.dae
- link head_tilt_link: geometry collision mesh filename=package://pr2_description/meshes/head_v0/head_tilt_L.stl; visual mesh filename=package://pr2_description/meshes/head_v0/head_tilt.dae
- link l_elbow_flex_link: geometry collision mesh filename=package://pr2_description/meshes/upper_arm_v0/elbow_flex.stl; visual mesh filename=package://pr2_description/meshes/upper_arm_v0/elbow_flex.dae
- link l_forearm_link: geometry collision mesh filename=package://pr2_description/meshes/forearm_v0/forearm.stl; visual mesh filename=package://pr2_description/meshes/forearm_v0/forearm.dae
- link l_gripper_l_finger_link: geometry collision mesh filename=package://pr2_description/meshes/gripper_v0/l_finger.stl; visual mesh filename=package://pr2_description/meshes/gripper_v0/l_finger.dae
- link l_gripper_l_finger_tip_link: geometry collision mesh filename=package://pr2_description/meshes/gripper_v0/l_finger_tip.stl; visual mesh filename=package://pr2_description/meshes/gripper_v0/l_finger_tip.dae
- link l_gripper_palm_link: geometry collision mesh filename=package://pr2_description/meshes/gripper_v0/gripper_palm.stl; visual mesh filename=package://pr2_description/meshes/gripper_v0/gripper_palm.dae
- link l_gripper_r_finger_link: geometry collision mesh filename=package://pr2_description/meshes/gripper_v0/l_finger.stl; visual mesh filename=package://pr2_description/meshes/gripper_v0/l_finger.dae
- link l_gripper_r_finger_tip_link: geometry collision mesh filename=package://pr2_description/meshes/gripper_v0/l_finger_tip.stl; visual mesh filename=package://pr2_description/meshes/gripper_v0/l_finger_tip.dae
- link l_shoulder_pan_link: geometry collision mesh filename=package://pr2_description/meshes/shoulder_v0/shoulder_pan.s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; visual mesh filename=package://pr2_description/meshes/shoulder_v0/shoulder_pan.d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
- link l_upper_arm_link: geometry collision mesh filename=package://pr2_description/meshes/upper_arm_v0/upper_arm.stl; visual mesh filename=package://pr2_description/meshes/upper_arm_v0/upper_arm.dae
- link l_wrist_flex_link: geometry collision mesh filename=package://pr2_description/meshes/forearm_v0/wrist_flex.stl; visual mesh filename=package://pr2_description/meshes/forearm_v0/wrist_flex.dae
- link r_elbow_flex_link: geometry collision mesh filename=package://pr2_description/meshes/upper_arm_v0/elbow_flex.stl; visual mesh filename=package://pr2_description/meshes/upper_arm_v0/elbow_flex.dae
- link r_forearm_link: geometry collision mesh filename=package://pr2_description/meshes/forearm_v0/forearm.stl; visual mesh filename=package://pr2_description/meshes/forearm_v0/forearm.dae
- link r_gripper_l_finger_link: geometry collision mesh filename=package://pr2_description/meshes/gripper_v0/l_finger.stl; visual mesh filename=package://pr2_description/meshes/gripper_v0/l_finger.dae
- link r_gripper_l_finger_tip_link: geometry collision mesh filename=package://pr2_description/meshes/gripper_v0/l_finger_tip.stl; visual mesh filename=package://pr2_description/meshes/gripper_v0/l_finger_tip.dae
- link r_gripper_palm_link: geometry collision mesh filename=package://pr2_description/meshes/gripper_v0/gripper_palm.stl; visual mesh filename=package://pr2_description/meshes/gripper_v0/gripper_palm.dae
- link r_gripper_r_finger_link: geometry collision mesh filename=package://pr2_description/meshes/gripper_v0/l_finger.stl; visual mesh filename=package://pr2_description/meshes/gripper_v0/l_finger.dae
- link r_gripper_r_finger_tip_link: geometry collision mesh filename=package://pr2_description/meshes/gripper_v0/l_finger_tip.stl; visual mesh filename=package://pr2_description/meshes/gripper_v0/l_finger_tip.dae
- link r_shoulder_pan_link: geometry collision mesh filename=package://pr2_description/meshes/shoulder_v0/shoulder_pan.s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; visual mesh filename=package://pr2_description/meshes/shoulder_v0/shoulder_pan.d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
- link r_upper_arm_link: geometry collision mesh filename=package://pr2_description/meshes/upper_arm_v0/upper_arm.stl; visual mesh filename=package://pr2_description/meshes/upper_arm_v0/upper_arm.dae
- link r_wrist_flex_link: geometry collision mesh filename=package://pr2_description/meshes/forearm_v0/wrist_flex.stl; visual mesh filename=package://pr2_description/meshes/forearm_v0/wrist_flex.dae
- link torso_lift_link: geometry collision mesh filename=package://pr2_description/meshes/torso_v0/torso_lift_L.stl; visual mesh filename=package://pr2_description/meshes/torso_v0/torso_lift.dae

File: ur10/ur10.urdf (robot description, URDF)
Before this commit: robot ur10, 9 links, 8 joints
Links:
- link base_link: geometry collision mesh filename=package://ur_description/meshes/ur10/collision/Base.stl; visual mesh filename=package://ur_description/meshes/ur10/visual/base.dae
- link forearm_link: geometry collision mesh filename=package://ur_description/meshes/ur10/collision/Forearm.stl; visual mesh filename=package://ur_description/meshes/ur10/visual/forearm.dae
- link shoulder_link: geometry collision mesh filename=package://ur_description/meshes/ur10/collision/Shoulder.stl; visual mesh filename=package://ur_description/meshes/ur10/visual/shoulder.dae
- link upper_arm_link: geometry collision mesh filename=package://ur_description/meshes/ur10/collision/UpperArm.stl; visual mesh filename=package://ur_description/meshes/ur10/visual/upperarm.dae
- link wrist_1_link: geometry collision mesh filename=package://ur_description/meshes/ur10/collision/Wrist1.stl; visual mesh filename=package://ur_description/meshes/ur10/visual/wrist1.dae
- link wrist_2_link: geometry collision mesh filename=package://ur_description/meshes/ur10/collision/Wrist2.stl; visual mesh filename=package://ur_description/meshes/ur10/visual/wrist2.dae
- link wrist_3_link: geometry collision mesh filename=package://ur_description/meshes/ur10/collision/Wrist3.stl; visual mesh filename=package://ur_description/meshes/ur10/visual/wrist3.dae
